File: Schematic/PCB Design/PCB Design.sch (KiCad schematic (older format))
At the start: 1 part

Commit message: initiated rev 2A of the board design
Parts:
- added J1: DHT11, PCB Design:conn_01x01, symbol Connector_Generic:Conn_01x01
- added J2: 3..3V Out, PCB Design:conn_01x01, symbol Connector_Generic:Conn_01x01
- added J3: RX/TX, PCB Design:conn_01x02, symbol Connector_Generic:Conn_01x02
- added J4: TrigSendPins, PCB Design:conn_01x08, symbol Connector_Generic:Conn_01x08
- added J5: EchoReturnPins, PCB Design:conn_01x08, symbol Connector_Generic:Conn_01x08
- added J6: Conn_01x04, PCB Design:conn_01x04, symbol Connector_Generic:Conn_01x04
- added SW1: SW_SPST, symbol Switch:SW_SPST
- added U1, U3: CD4051B, Package_DIP:DIP-16_W7.62mm, symbol Analog_Switch:CD4051B
- added U2: ESP32-CAM, PCB Design:ESP32CAM, symbol Project_Symbols:ESP32-CAM
Connections:
- net +3V3: now also J2.1 (Pin_1), U2.9 (3V3)
- net +5V: now also J6.1 (Pin_1), U1.16 (VDD), U2.8 (5V), U3.16 (VDD)
- net GND: now also J6.2 (Pin_2), SW1.2 (B), U1.6 (INH), U1.7 (VEE), U1.8 (VSS), U2.12 (GND), U2.16 (GND), U2.7 (GND), U3.6 (INH), U3.7 (VEE), U3.8 (VSS)
- new net: J1.1 (Pin_1), U2.1 (IO4)
- new net: J3.1 (Pin_1), U2.14 (U0R)
- new net: J3.2 (Pin_2), U2.15 (U0T)
- new net: J5.1 (Pin_1), U3.13 (X0)
- new net: J5.2 (Pin_2), U3.14 (X1)
- new net: J5.3 (Pin_3), U3.15 (X2)
- new net: J5.4 (Pin_4), U3.12 (X3)
- new net: J5.5 (Pin_5), U3.1 (X4)
- new net: J5.6 (Pin_6), U3.5 (X5)
- new net: J5.7 (Pin_7), U3.2 (X6)
- new net: J5.8 (Pin_8), U3.4 (X7)
- new net: J4.1 (Pin_1), U1.13 (X0)
- new net: J4.2 (Pin_2), U1.14 (X1)
- new net: J4.3 (Pin_3), U1.15 (X2)
- new net: J4.4 (Pin_4), U1.12 (X3)
- new net: J4.5 (Pin_5), U1.1 (X4)
- new net: J4.6 (Pin_6), U1.5 (X5)
- new net: J4.7 (Pin_7), U1.2 (X6)
- new net: J4.8 (Pin_8), U1.4 (X7)
- new net displayCLA: J6.3 (Pin_3), U2.6 (IO12)
- new net displaySDA: J6.4 (Pin_4), U2.5 (IO13)
- new net echoSignal: U2.10 (IO16), U3.3 (X)
- new net enable: SW1.1 (A), U1.3 (X), U2.11 (IO0)
- new net selectA: U1.11 (A), U2.4 (IO15), U3.11 (A)
- new net selectB: U1.10 (B), U2.3 (IO14), U3.10 (B)
- new net selectC: U1.9 (C), U2.2 (IO2), U3.9 (C)
- no-connect marks 0 -> 1
Other:
- note added: "Signals recieved from\nECHO pin on HC-SR04"
- note added: "Signals to be sent to\nTRIG pin on HC-SR04"
